Commit message: Fixed depth camera issue

File: husky_description/urdf/accessories/husky_rgbdcamera.urdf.xacro (robot description, xacro)
@@ -26,4 +26,5 @@
     </inertial>
   </link>
+  <link name="front_rgbd_optical_frame"></link>
   <joint name="front_rgbd_joint" type="fixed">
     <parent link="base_link"/>
@@ -31,7 +32,13 @@
     <origin xyz="0.0 0.0 0.45" rpy="0 0 0"/>
   </joint>
+  <joint name="front_rgbd_optical_joint" type="fixed">
+    <parent link="front_rgbd_frame"/>
+    <child link="front_rgbd_optical_frame"/>
+    <origin xyz="0 0 0" rpy="-1.5708 0 0"/>
+  </joint>
   <gazebo reference="front_rgbd_frame">
-    <sensor name="front_rgbd" type="camera">
-      <update_rate>30</update_rate>
+    <sensor name="camera" type="depth">
+      <pose> 0 0 0 0 0 0 </pose>
+      <update_rate>20</update_rate>
       <camera>
         <horizontal_fov>1.3962634</horizontal_fov>
@@ -46,23 +53,6 @@
         </clip>
       </camera>
-      <!-- <depth_camera>
-        <clip>
-          <near>0.1</near>
-          <far>3.0</far>
-        </clip>
-      </depth_camera> -->
       <plugin name="camera_controller" filename="libgazebo_ros_camera.so">
-        <alwaysOn>true</alwaysOn>
-        <updateRate>0.0</updateRate>
-        <cameraName>front_rgbd</cameraName>
-        <imageTopicName>image_raw</imageTopicName>
-        <cameraInfoTopicName>camera_info</cameraInfoTopicName>
-        <frameName>front_rgbd_frame</frameName>
-        <hackBaseline>0.07</hackBaseline>
-        <distortionK1>0.0</distortionK1>
-        <distortionK2>0.0</distortionK2>
-        <distortionK3>0.0</distortionK3>
-        <distortionT1>0.0</distortionT1>
-        <distortionT2>0.0</distortionT2>
+        <frame_name>front_rgbd_optical_frame</frame_name>
       </plugin>
     </sensor>

Commit message: Fixed the transformation between the camera link and the base link

File: husky_description/urdf/accessories/husky_rgbdcamera.urdf.xacro (robot description, xacro)
@@ -35,10 +35,10 @@
     <parent link="front_rgbd_frame"/>
     <child link="front_rgbd_optical_frame"/>
-    <origin xyz="0 0 0" rpy="-1.5708 0 0"/>
+    <origin xyz="0 0 0" rpy="-1.5708 0 -1.5708"/>
   </joint>
   <gazebo reference="front_rgbd_frame">
     <sensor name="camera" type="depth">
       <pose> 0 0 0 0 0 0 </pose>
-      <update_rate>20</update_rate>
+      <update_rate>10</update_rate>
       <camera>
         <horizontal_fov>1.3962634</horizontal_fov>
@@ -50,5 +50,5 @@
         <clip>
           <near>0.1</near>
-          <far>3.0</far>
+          <far>5.0</far>
         </clip>
       </camera>
